File: aquaponics_pcb/aquaponics_pcb/_autosave-aquaponics_pcb.kicad_pcb (KiCad board)
At the start: 2 copper layers, 60.5 x 73.5 mm, 67 parts, among them IC1 AZ1117CH-3.3TRG1, IC2 ESP32-S3-WROOM-1U-N8, IC3 ADM3260ARSZ, IC4 DRV8214RTER, IC5 DRV8214RTER, J1 RFPC-SMA27-F, J2 2338792-1, J3 RFPC-SMA27-F, J4 RFPC-SMA27-F, J5 Screw_Terminal_01x02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

Commit message: finish ground and power pours. fix rules and run final DRC. export gerbers
Connections:
- net +3V3 renamed V_MCU
